Commit message: fix: rpy

File: config/lekiwi.ros2_control.xacro (robot description, xacro)
@@ -14,5 +14,5 @@
                 </xacro:unless>
             </hardware>
-            <joint name="ST3215_Servo_Motor-v1-2_Revolute-60">
+            <joint name="joint7">
                 <command_interface name="velocity"/>
                 <state_interface name="position">
@@ -21,6 +21,8 @@
                 <state_interface name="velocity"/>
                 <param name="motor_id">7</param>
+                <param name="direction">-1</param>
+                <param name="control_mode">velocity</param>
             </joint>
-            <joint name="ST3215_Servo_Motor-v1-1_Revolute-62">
+            <joint name="joint8">
                 <command_interface name="velocity"/>
                 <state_interface name="position">
@@ -29,6 +31,8 @@
                 <state_interface name="velocity"/>
                 <param name="motor_id">8</param>
+                <param name="direction">-1</param>
+                <param name="control_mode">velocity</param>
             </joint>
-            <joint name="ST3215_Servo_Motor-v1_Revolute-64">
+            <joint name="joint9">
                 <command_interface name="velocity"/>
                 <state_interface name="position">
@@ -37,4 +41,6 @@
                 <state_interface name="velocity"/>
                 <param name="motor_id">9</param>
+                <param name="direction">-1</param>
+                <param name="control_mode">velocity</param>
             </joint>
         </ros2_control>

File: urdf/lekiwi.urdf (robot description, URDF)
Before this commit: robot LeKiwi, 46 links, 45 joints
Joints:
- removed joint ST3215_Servo_Motor-v1-1_Revolute-62
- removed joint ST3215_Servo_Motor-v1-2_Revolute-60
- removed joint ST3215_Servo_Motor-v1_Revolute-64
- added joint joint7: type continuous, parent ST3215_Servo_Motor-v1, child omni_wheel_mount-v5, origin xyz=0.010249999999999999 -0.010762340000000004 0.046859090000000006 rpy=-1.5707963267948966 1.5707963267948966 0, axis -0.866025 -2.0578792567370943e-32 0.5
- added joint joint8: type continuous, parent ST3215_Servo_Motor-v1-2, child omni_wheel_mount-v5-2, origin xyz=0.010249999999999999 -0.035199999999999995 -0.03275 rpy=-1.5707963267948966 1.5707963267948966 0, axis 0.0 0.0 -1.0
- added joint joint9: type continuous, parent ST3215_Servo_Motor-v1-1, child omni_wheel_mount-v5-1, origin xyz=0.010249999999999999 0.04636234 -0.014801910000000005 rpy=-1.5707963267948966 1.5707963267948966 0, axis 0.866025 1.0674582272562919e-32 0.5
- joint base_mount: origin (none) -> xyz=0.0 0.0 0.0 rpy=0.0 0.0 -1.5707963267948966
